Commit message: working dishwasher controller upper basket

File: dishwasher_description/urdf/dishwasher.urdf (robot description, URDF)
Before this commit: robot dishwasher, 4 links, 3 joints
Links:
- link base_link: geometry collision mesh filename=package://dishwasher_description/meshes/base_link.STL; visual mesh filename=package://dishwasher_description/meshes/base_link.STL
- link door_link: geometry collision mesh filename=package://dishwasher_description/meshes/door_link.STL; visual mesh filename=package://dishwasher_description/meshes/door_link.STL
- link lower_basket_link: geometry collision mesh filename=package://dishwasher_description/meshes/lower_basket_link.S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; visual mesh filename=package://dishwasher_description/meshes/lower_basket_link.S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
- link upper_basket_link: geometry collision mesh filename=package://dishwasher_description/meshes/upper_basket_link.S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; visual mesh filename=package://dishwasher_description/meshes/upper_basket_link.S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
Joints:
- joint upper_basket_joint: limit lower=0 upper=0 effort=0 velocity=0 -> lower=-0.1 upper=0.1 effort=10 velocity=10

Commit message: working dishwasher with texture and upper and lower basket controller

File: dishwasher_description/urdf/dishwasher.urdf (robot description, URDF)
Before this commit: robot dishwasher, 4 links, 3 joints
Joints:
- joint lower_basket_joint: limit lower=0 upper=0 effort=0 velocity=0 -> lower=-0.1 upper=0.6 effort=10 velocity=10
- joint upper_basket_joint: limit lower=-0.1 upper=0.1 effort=10 velocity=10 -> lower=-0.1 upper=0.4 effort=10 velocity=10
